File: A-BRIDGE.sch (EAGLE design)
At the start: 10 parts, among them IC1 74HC240DW, IC2 A4950, IC3 A4950

Commit message: rev2.01
Added "hot surface" warning
Better heat dissipation on bottom area
Bigger capacitor's footprint for hand soldering
Parts:
- C1, C2: device rcl:CPOL-EUUD-6,3X7,7 -> rcl:CPOL-EUUD-6,3X7,7-HS
Changed lines of the file:
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@@
 <part name="SV1" library="con-lsta" deviceset="FE06-1" device=""/>
 <part name="SV2" library="con-lsta" deviceset="FE06-1" device=""/>
-<part name="C1" library="rcl" deviceset="CPOL-EU" device="UD-6,3X7,7" value="100u"/>
-<part name="C2" library="rcl" deviceset="CPOL-EU" device="UD-6,3X7,7" value="100u"/>
+<part name="C1" library="rcl" deviceset="CPOL-EU" device="UD-6,3X7,7-HS" value="100u"/>
+<part name="C2" library="rcl" deviceset="CPOL-EU" device="UD-6,3X7,7-HS" value="100u"/>
 <part name="C3" library="rcl" deviceset="C-EU" device="C0805K" value="220n"/>
 <part name="C4" library="rcl" deviceset="C-EU" device="C0805K" value="220n"/>
